File: pcb/pico_expansion_board.kicad_sch (KiCad schematic)
At the start: 53 parts, among them IC1 TPS5450DDA, J1 DC12V/24V, J10 CAN_L, J2 TMC2209 Motor 1, J3 TMC2209 Motor 2, J4 Motor 1, J5 Motor 2, J6 Straight Through, J7 NULL Modem, J8 EXP1, J9 EXP2, SW1 SW_Push, U1 MAX232, U2 MCP2542FDxMF, U3 Pico, U5 CAT24C256

Commit message: Update to v3
Parts:
- removed C2, C3: 100nF, Capacitor_SMD:C_0805_2012Metric, symbol Device:C
- removed J10: CAN_L, TerminalBlock:TerminalBlock_bornier-2_P5.08mm, symbol Connector:Screw_Terminal_01x02
- removed J7: NULL Modem, Connector_Dsub:DSUB-9_Male_Horizontal_P2.77x2.84mm_EdgePinOffset7.70mm_Housed_MountingHolesOffset9.12mm, symbol Connector:DE9_Receptacle_MountingHoles
- removed JP9: 120JP, Connector_PinHeader_2.00mm:PinHeader_1x02_P2.00mm_Vertical, symbol Jumper:Jumper_2_Open
- removed R1: 120Ω, Resistor_SMD:R_0805_2012Metric, symbol Device:R
- removed TP5: TestPoint, TestPoint:TestPoint_Pad_2.0x2.0mm, symbol Connector:TestPoint
- removed U1: MAX232, Package_SO:SOIC-16_3.9x9.9mm_P1.27mm, symbol Interface_UART:MAX232
- removed U2: MCP2542FDxMF, Package_SO:SO-8_3.9x4.9mm_P1.27mm, symbol Interface_CAN_LIN:MCP2542FDxMF
- added C14: 0.1uF, Capacitor_SMD:C_0805_2012Metric_Pad1.18x1.45mm_HandSolder, symbol Device:C
- added C15, C16: 10nF, Capacitor_SMD:C_0805_2012Metric_Pad1.18x1.45mm_HandSolder, symbol Device:C
- added D2: GREEN, Diode_SMD:D_0805_2012Metric_Pad1.15x1.40mm_HandSolder, symbol Device:LED
- added D3, D4: RED, Diode_SMD:D_0805_2012Metric_Pad1.15x1.40mm_HandSolder, symbol Device:LED
- added JP5, JP6, JP7: ~, Connector_PinSocket_2.00mm:PinSocket_1x03_P2.00mm_Vertical, symbol Jumper:Jumper_3_Bridged12
- added R3, R5: 10K, Resistor_SMD:R_0805_2012Metric_Pad1.20x1.40mm_HandSolder, symbol Device:R
- added R6, R9: 4.7k, Resistor_SMD:R_0805_2012Metric_Pad1.20x1.40mm_HandSolder, symbol Device:R
- added R7: 300, Resistor_SMD:R_0805_2012Metric_Pad1.20x1.40mm_HandSolder, symbol Device:R
- added R8: 680, Resistor_SMD:R_0805_2012Metric_Pad1.20x1.40mm_HandSolder, symbol Device:R
- added U1: MAX3232, Package_SO:SOIC-16_3.9x9.9mm_P1.27mm, symbol Interface_UART:MAX3232
- added U4: 74LVC1G125, Package_TO_SOT_SMD:SOT-353_SC-70-5_Handsoldering, symbol 74xGxx:74LVC1G125
- added U5: AMS1117-3.3, Package_TO_SOT_SMD:SOT-223-3_TabPin2, symbol Regulator_Linear:AMS1117-3.3
- C1: renamed from C5; footprint Capacitor_SMD:C_0805_2012Metric -> Capacitor_SMD:C_0805_2012Metric_Pad1.18x1.45mm_HandSolder
- C10: renamed from C17; footprint Capacitor_SMD:C_0805_2012Metric -> Capacitor_SMD:C_0805_2012Metric_Pad1.18x1.45mm_HandSolder
- C11: renamed from C8; value 10uF -> 0.1uF; footprint Capacitor_SMD:C_0805_2012Metric -> Capacitor_SMD:C_0805_2012Metric_Pad1.18x1.45mm_HandSolder
- C13: renamed from C19; footprint Capacitor_SMD:C_0805_2012Metric -> Capacitor_SMD:C_0805_2012Metric_Pad1.18x1.45mm_HandSolder
- C2: renamed from C1; value 1uF -> 0.1uF; footprint Capacitor_SMD:C_0805_2012Metric -> Capacitor_SMD:C_0805_2012Metric_Pad1.18x1.45mm_HandSolder
- C3: renamed from C9; footprint Capacitor_SMD:C_0805_2012Metric -> Capacitor_SMD:C_0805_2012Metric_Pad1.18x1.45mm_HandSolder
- C4: renamed from C16; footprint Capacitor_SMD:C_0805_2012Metric -> Capacitor_SMD:C_0805_2012Metric_Pad1.18x1.45mm_HandSolder
- C5: renamed from C4; value 1uF -> 0.1uF; footprint Capacitor_SMD:C_0805_2012Metric -> Capacitor_SMD:C_0805_2012Metric_Pad1.18x1.45mm_HandSolder
- C6: value 1uF -> 0.1uF; footprint Capacitor_SMD:C_0805_2012Metric -> Capacitor_SMD:C_0805_2012Metric_Pad1.18x1.45mm_HandSolder
- C7: value 10uF -> 0.1uF; footprint Capacitor_SMD:C_0805_2012Metric -> Capacitor_SMD:C_0805_2012Metric_Pad1.18x1.45mm_HandSolder
- D1: footprint DO-214AC -> Diode_SMD:D_SMA
- H1, H2, H3, H4: value MountingHole -> ~
- J6: value Straight Through -> ~
- R1: renamed from R2; footprint Resistor_SMD:R_0805_2012Metric -> Resistor_SMD:R_0805_2012Metric_Pad1.20x1.40mm_HandSolder
- R2: renamed from R6; footprint Resistor_SMD:R_0805_2012Metric -> Resistor_SMD:R_0805_2012Metric_Pad1.20x1.40mm_HandSolder
- R4: renamed from R3; footprint Resistor_SMD:R_0805_2012Metric -> Resistor_SMD:R_0805_2012Metric_Pad1.20x1.40mm_HandSolder
- TP1: renamed from TP6; value TestPoint -> ~
- TP2: renamed from TP7; value TestPoint -> ~
- TP3: renamed from TP8; value TestPoint -> ~
- TP4: renamed from TP1; value TestPoint -> ~
- TP5: renamed from TP2; value TestPoint -> ~
- renumbered C18 to C12, C11 to C8, C12 to C9, TP4 to TP_UART1, U3 to U2, U5 to U3
Connections:
- net +3.3V: now also C5.1, J2.15 (VDD), J3.15 (VDD), J3.7 (MS1), U3.8 (VCC), JP7.2 (C), R3.1, R5.1, U1.16 (VCC); no longer U2.36 (3V3)
- net +5V: now also C14.1, C16.1, R8.2, U4.5 (VCC), U5.3 (VI); no longer C11.2, C5.1, J2.15 (VDD), J3.15 (VDD), J3.7 (MS1), U3.8 (VCC)
- net EEPROM_SCL: now also R5.2
- net EEPROM_SDA: now also R3.2
- net GND: now also C11.2, C14.2, C15.2, C16.2, D2.1 (K), D3.1 (K), D4.1 (K), R6.2, U1.15 (GND), U4.1, U4.3 (GND), U5.1 (GND); no longer J2.3 (CLK), J3.3 (CLK)
- net MOTOR_UART: now also JP1.2 (B), JP3.2 (B); no longer JP1.1 (A), JP3.1 (A)
- net NEOPIXEL: now also U2.17 (GPIO13), R6.1, U4.2; no longer J8.6 (Pin_6), U2.31 (GPIO26_ADC0)
- net SCALE_RXD: now also JP6.2 (C), U1.13 (R1IN); no longer J6.2
- net SCALE_TXD: now also JP5.2 (C), U1.14 (T1OUT); no longer J6.3
- net SCALE_UART_RX: now also U1.12 (R1OUT)
- net SCALE_UART_TX: now also U1.11 (T1IN)
- net VCC: now also R9.2
- net at J3.4 (PDN): now also JP3.1 (A); no longer JP3.2 (B)
- net at J2.4 (PDN): now also JP1.1 (A); no longer JP1.2 (B)
- net at C11.1: now also U1.2 (VS+)
- net at C7.2: now also U1.6 (VS-)
- net at C2.1: now also U1.1 (C1+)
- net at C2.2: now also U1.3 (C1-)
- net at C6.1: now also U1.4 (C2+)
- net at C6.2: now also U1.5 (C2-)
- net CAN_RX: no longer names the net of U2.34 (GPIO28_ADC2)
- net CAN_TX: no longer names the net of U2.32 (GPIO27_ADC1)
- new net: D3.2 (A), R8.1
- new net: D2.2 (A), R7.1
- new net: D4.2 (A), R9.1
- new net 3.3V_PICO: JP7.3 (B), U2.36 (3V3)
- new net 3.3V_REG: C15.1, JP7.1 (A), R7.2, U5.2 (VO)
- new net NEOPIXEL_5V: J8.6 (Pin_6), U4.4
- new net RS232_PIN2: J6.2, JP5.1 (A), JP6.3 (B)
- new net RS232_PIN3: J6.3, JP5.3 (B), JP6.1 (A)
- no-connect marks 33 -> 31
Other:
- note added: "3.3V power selector"
- note added: "NULL Modem and Straight Through Select"
- note added: "NeoPixel RGB LED Level Converter"
- note added: "Power Supply 3.3V out"
- note added: "Power Supply 5V out"
- note added: "Status LEDs"
- note removed: "CAN Transceiver"
- note removed: "Power Supply"
- moved on the sheet: C1, C10, C11, C12, C13, C2, C3, C4, C5, C6, C7, C8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

Commit message: Update v0.3 PCB
Parts:
- removed JP1: M1_UART_OP1, Connector_PinHeader_2.00mm:PinHeader_1x02_P2.00mm_Vertical, symbol Jumper:Jumper_2_Open
- removed JP2: M1_UART_OP2, Connector_PinHeader_2.00mm:PinHeader_1x02_P2.00mm_Vertical, symbol Jumper:Jumper_2_Open
- removed JP3: M2_UART_OP1, Connector_PinSocket_2.00mm:PinSocket_1x02_P2.00mm_Vertical, symbol Jumper:Jumper_2_Open
- removed JP4: M2_UART_OP2, Connector_PinSocket_2.00mm:PinSocket_1x02_P2.00mm_Vertical, symbol Jumper:Jumper_2_Open
- D1: footprint Diode_SMD:D_SMA -> DO-214AC
- J2, J3: footprint fab:Conn_StepStick -> Extra Footprints:Conn_StepStick_smaller_hole
- TP_UART1: value TestPoint -> ~
- U4: footprint Package_TO_SOT_SMD:SOT-353_SC-70-5_Handsoldering -> Package_TO_SOT_SMD:SOT-23-5
Connections:
- net MOTOR_UART: now also J2.5 (UART), J3.5 (UART)
- net PH_NET: now reaches C10.2, D1.C, IC1.8 (PH), L1.1
- no-connect marks 31 -> 33
Other:
- moved on the sheet: TP_UART1
