File: pcb/pico_expansion_board.kicad_sch (KiCad schematic)
At the start: 57 parts, among them IC1 TPS5450DDA, J1 DC12V/24V, J2 TMC2209 Motor 1, J3 TMC2209 Motor 2, J4 Motor 1, J5 Motor 2, J8 EXP1, J9 EXP2, SW1 SW_Push, U1 MAX3232, U2 Pico, U3 CAT24C256, U4 74LVC1G125, U5 AMS1117-3.3

Commit message: Update 3D model mapping, fix the footprint for jumpers
Parts:
- JP5, JP6, JP7: footprint Connector_PinSocket_2.00mm:PinSocket_1x03_P2.00mm_Vertical -> Connector_PinHeader_2.00mm:PinHeader_1x03_P2.00mm_Vertical
Changed lines of the file:
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@@
       (effects (font (size 1.27 1.27)) (justify left))
     )
-    (property "Footprint" "Connector_PinSocket_2.00mm:PinSocket_1x03_P2.00mm_Vertical" (at 320.04 104.14 0)
+    (property "Footprint" "Connector_PinHeader_2.00mm:PinHeader_1x03_P2.00mm_Vertical" (at 320.04 104.14 0)
       (effects (font (size 1.27 1.27)) hide)
     )
@@
       (effects (font (size 1.27 1.27)) (justify left))
     )
-    (property "Footprint" "Connector_PinSocket_2.00mm:PinSocket_1x03_P2.00mm_Vertical" (at 320.04 120.65 0)
+    (property "Footprint" "Connector_PinHeader_2.00mm:PinHeader_1x03_P2.00mm_Vertical" (at 320.04 120.65 0)
       (effects (font (size 1.27 1.27)) hide)
     )
@@
       (effects (font (size 1.27 1.27)) (justify left))
     )
-    (property "Footprint" "Connector_PinSocket_2.00mm:PinSocket_1x03_P2.00mm_Vertical" (at 105.41 190.5 0)
-      (effects (font (size 1.27 1.27)) hide)
-    )
+    (property "Footprint" "Connector_PinHeader_2.00mm:PinHeader_1x03_P2.00mm_Vertical" (at 105.41 190.5 0)
+      (effects (font (size 1.27 1.27)) hide)
+    )

Commit message: Fix the bug where Pin 5 from RS232 was not connected to the ground, update several labels
Connections:
- net GND: now also J6.5
- no-connect marks 33 -> 32
Changed lines of the file:
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@@
   (junction (at 46.99 204.47) (diameter 0) (color 0 0 0 0)
+  )
+  (junction (at 383.54 129.54) (diameter 0) (color 0 0 0 0)
   )
   (junction (at 22.86 124.46) (diameter 0) (color 0 0 0 0)
@@
   (no_connect (at 375.92 115.57))
   (no_connect (at 247.65 58.42))
-  (no_connect (at 375.92 123.19))
   (no_connect (at 62.23 137.16))
   (no_connect (at 76.2 90.17))
@@
     (stroke (width 0) (type default))
   )
+  (wire (pts (xy 383.54 132.08) (xy 383.54 129.54))
+    (stroke (width 0) (type default))
+  )
   (wire (pts (xy 76.2 261.62) (xy 76.2 264.16))
     (stroke (width 0) (type default))
@@
     (stroke (width 0) (type default))
   )
+  (wire (pts (xy 375.92 129.54) (xy 383.54 129.54))
+    (stroke (width 0) (type default))
+  )
   (wire (pts (xy 252.73 184.15) (xy 280.67 184.15))
     (stroke (width 0) (type default))
@@
     (stroke (width 0) (type default))
   )
+  (wire (pts (xy 375.92 123.19) (xy 375.92 129.54))
+    (stroke (width 0) (type default))
+  )
   (wire (pts (xy 312.42 241.3) (xy 323.85 241.3))
     (stroke (width 0) (type default))
@@
   )
   (wire (pts (xy 214.63 142.24) (xy 214.63 144.78))
+    (stroke (width 0) (type default))
+  )
+  (wire (pts (xy 383.54 129.54) (xy 383.54 128.27))
     (stroke (width 0) (type default))
   )
@@
     )
   )
-  (symbol (lib_id "power:GND") (at 383.54 128.27 0) (unit 1)
-    (in_bom yes) (on_board yes) (dnp no) (fields_autoplaced)
-    (property "Reference" "#PWR025" (at 383.54 134.62 0)
-      (effects (font (size 1.27 1.27)) hide)
-    )
-    (property "Value" "GND" (at 383.54 133.35 0)
-      (effects (font (size 1.27 1.27)))
-    )
-    (property "Footprint" "" (at 383.54 128.27 0)
-      (effects (font (size 1.27 1.27)) hide)
-    )
-    (property "Datasheet" "" (at 383.54 128.27 0)
-      (effects (font (size 1.27 1.27)) hide)
-    )
+  (symbol (lib_id "power:GND") (at 383.54 132.08 0) (unit 1)
+    (in_bom yes) (on_board yes) (dnp no) (fields_autoplaced)
+    (property "Reference" "#PWR025" (at 383.54 138.43 0)
+      (effects (font (size 1.27 1.27)) hide)
+    )
+    (property "Value" "GND" (at 383.54 137.16 0)
+      (effects (font (size 1.27 1.27)))
+    )
+    (property "Footprint" "" (at 383.54 132.08 0)
+      (effects (font (size 1.27 1.27)) hide)
+    )
+    (property "Datasheet" "" (at 383.54 132.08 0)
+      (effects (font (size 1.27 1.27)) hide)
+    )
