File: pcb/pico_expansion_board.kicad_pcb (KiCad board)
At the start: 4 copper layers, 91.7 x 66.8 mm, 57 parts, among them IC1 TPS5450DDA, J1 DC12V/24V, J2 TMC2209 Motor 1, J3 TMC2209 Motor 2, J4 Motor 1, J5 Motor 2, J8 EXP1, J9 EXP2, SW1 SW_Push, U1 MAX3232, U2 Pico, U3 CAT24C256, U4 74LVC1G125, U5 AMS1117-3.3

Commit message: Up-rev to v1.0 release
Other:
- board text added: "OpenTrickler Controller v1.0"
- board text removed: "OpenTrickler Controller v1.0rc"
Changed lines of the file:
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@@
     (effects (font (size 1 1) (thickness 0.125)) (justify left bottom mirror))
   )
-  (gr_text "OpenTrickler Controller v1.0rc" (at 98.298 75.946) (layer "B.SilkS")
+  (gr_text "OpenTrickler Controller v1.0" (at 98.298 75.946) (layer "B.SilkS")
     (effects (font (size 1 1) (thickness 0.1875)) (justify left bottom mirror))
   )
@@
     (effects (font (size 0.8 0.8) (thickness 0.1)) (justify left bottom))
   )
-  (gr_text "OpenTrickler Controller v1.0rc" (at 77.216 75.946) (layer "F.SilkS")
+  (gr_text "OpenTrickler Controller v1.0" (at 77.216 75.946) (layer "F.SilkS")
     (effects (font (size 1 1) (thickness 0.1875)) (justify left bottom))
   )
