File: pwm_expansion_board/pcb/pwm_expansion_board.kicad_pcb (KiCad board)
At the start: 2 copper layers, 21.2 x 51.2 mm, 13 parts, among them J1 Conn_01x03_Pin, J2 Conn_01x03_Pin, J3 Conn_01x03_Pin, U1 Pico, U2 74LVC1G125, U3 74LVC1G125, U4 74LVC1G125

Commit message: Improve GND via
Routing:
- net GND: track 6.23 -> 0.04 mm, vias 10 -> 12
Changed lines of the file:
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@@
-	)
-	(segment
-		(start 139.7 59.2)
-		(end 138.75 58.25)
-		(width 0.5)
-		(layer "F.Cu")
-		(net 2)
-	)
-	(segment
-		(start 137.7125 57.2125)
-		(end 138.75 58.25)
-		(width 0.5)
-		(layer "F.Cu")
-		(net 2)
-	)
-	(segment
-		(start 139.7 59.8625)
-		(end 139.7 59.2)
-		(width 0.5)
-		(layer "F.Cu")
-		(net 2)
-	)
-	(segment
-		(start 137.7125 56.5)
-		(end 137.7125 57.2125)
-		(width 0.5)
-		(layer "F.Cu")
-		(net 2)
-	)
-	(segment
-		(start 137.8 59.2)
-		(end 137.8 59.8625)
-		(width 0.5)
-		(layer "F.Cu")
-		(net 2)
 	)
 	(segment
 		(start 137.7125 102)
 		(end 137.75 102)
-		(width 0.5)
-		(layer "F.Cu")
-		(net 2)
-	)
-	(segment
-		(start 138.75 58.25)
-		(end 137.8 59.2)
 		(width 0.5)
 		(layer "F.Cu")
@@
 	)
 	(via
-		(at 138.75 58.25)
-		(size 0.6)
-		(drill 0.3)
-		(layers "F.Cu" "B.Cu")
-		(net 2)
-	)
-	(via
 		(at 137.8 96.3625)
 		(size 0.6)
@@
 	(via
 		(at 139.75 64.25)
+		(size 0.6)
+		(drill 0.3)
+		(layers "F.Cu" "B.Cu")
+		(net 2)
+	)
+	(via
+		(at 139.7 59.8625)
 		(size 0.6)
 		(drill 0.3)
@@
 		(size 0.6)
 		(drill 0.3)
+		(layers "F.Cu" "B.Cu")
+		(net 2)
+	)
+	(via
+		(at 137.8 59.8625)
+		(size 0.6)
+		(drill 0.3)
+		(layers "F.Cu" "B.Cu")
+		(net 2)
+	)
+	(via
+		(at 137.7125 56.5)
+		(size 0.6)
+		(drill 0.3)

Commit message: Add readme for pwm expansion board
Other:
- board text added: "OpenTrickler 5V PWM Expander Board Ver 1.0"
- board text removed: "OpenTrickler 5V PWM Expander Board Ver 0.1"
Changed lines of the file:
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@@
 		(layer "Edge.Cuts")
 	)
-	(gr_text "OpenTrickler\n5V PWM Expander Board\nVer 0.1"
+	(gr_text "OpenTrickler\n5V PWM Expander Board\nVer 1.0"
 		(at 140.208 53.086 90)
 		(layer "B.SilkS")
