File: motor_expansion_board_v2/pcb/rs232_transceiver.kicad_sch (KiCad schematic)
At the start: 12 parts, among them J8 Conn_02x02_Odd_Even, U4 MAX3232

Commit message: Add part numbers
Parts:
- C10: renamed from C11; LCSC Part # (none) -> C49678
- C11: renamed from C12; LCSC Part # (none) -> C49678
- C12: renamed from C13; LCSC Part # (none) -> C49678
- C13: renamed from C14; LCSC Part # (none) -> C49678
- C14: renamed from C15; LCSC Part # (none) -> C49678
- D5: LCSC Part # (none) -> C84256
- D6: LCSC Part # (none) -> C965817
- J10: renamed from J9; LCSC Part # (none) -> C426221; LCSC Part # (backup) (none) -> C141880
- J9: renamed from J8; LCSC Part # (none) -> C2935957; LCSC Part # (backup) (none) -> C2905988
- R11: renamed from R13; LCSC Part # (none) -> C17513
- R12: renamed from R14; LCSC Part # (none) -> C17513
- U4: LCSC Part # (none) -> C18261
Changed lines of the file:
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@@
 		(dnp no)
 		(fields_autoplaced yes)
-		(property "Reference" "#PWR053"
+		(property "Reference" "#PWR061"
 			(at 130.81 68.58 0)
 			(effects
@@
 			(project "pico_expansion_board"
 				(path "/b8f3f05d-f7a7-4c52-a258-9c2fea48c789/c872847a-864f-4ac1-95f5-557947400505"
-					(reference "#PWR053")
+					(reference "#PWR061")
 					(unit 1)
 				)
@@
 		(dnp no)
 		(fields_autoplaced yes)
-		(property "Reference" "C11"
+		(property "Reference" "C10"
 			(at 45.72 50.8 0)
 			(effects
@@
 			)
 		)
+		(property "LCSC Part #" "C49678"
+			(at 41.91 52.07 0)
+			(effects
+				(font
+					(size 1.27 1.27)
+				)
+				(hide yes)
+			)
+		)
 		(pin "1"
 		)
@@
 			(project "pico_expansion_board"
 				(path "/b8f3f05d-f7a7-4c52-a258-9c2fea48c789/c872847a-864f-4ac1-95f5-557947400505"
-					(reference "C11")
+					(reference "C10")
 					(unit 1)
 				)
@@
 		(dnp no)
 		(fields_autoplaced yes)
-		(property "Reference" "#PWR040"
+		(property "Reference" "#PWR059"
 			(at 80.01 34.29 0)
 			(effects
@@
 			(project "pico_expansion_board"
 				(path "/b8f3f05d-f7a7-4c52-a258-9c2fea48c789/c872847a-864f-4ac1-95f5-557947400505"
-					(reference "#PWR040")
+					(reference "#PWR059")
 					(unit 1)
 				)
@@
 			)
 		)
+		(property "LCSC Part #" "C18261"
+			(at 80.01 71.12 0)
+			(effects
+				(font
+					(size 1.27 1.27)
+				)
+				(hide yes)
+			)
+		)
 		(pin "1"
 		)
@@
 		(on_board yes)
 		(dnp no)
-		(property "Reference" "R14"
+		(property "Reference" "R12"
 			(at 207.01 105.41 0)
 			(effects
@@
 			)
 		)
+		(property "LCSC Part #" "C17513"
+			(at 201.93 106.68 0)
+			(effects
+				(font
+					(size 1.27 1.27)
+				)
+				(hide yes)
+			)
+		)
 		(pin "1"
 		)
@@
 			(project "pico_expansion_board"
 				(path "/b8f3f05d-f7a7-4c52-a258-9c2fea48c789/c872847a-864f-4ac1-95f5-557947400505"
-					(reference "R14")
+					(reference "R12")
 					(unit 1)
 				)
@@
 		(dnp no)
 		(fields_autoplaced yes)
-		(property "Reference" "#PWR052"
+		(property "Reference" "#PWR060"
 			(at 80.01 107.95 0)
 			(effects
@@
 			(project "pico_expansion_board"
 				(path "/b8f3f05d-f7a7-4c52-a258-9c2fea48c789/c872847a-864f-4ac1-95f5-557947400505"
-					(reference "#PWR052")
+					(reference "#PWR060")
 					(unit 1)
 				)
@@
 		(dnp no)
 		(fields_autoplaced yes)
-		(property "Reference" "J9"
+		(property "Reference" "J10"
 			(at 257.81 45.085 0)
 			(effects
@@
 			)
 		)
-		(property "Datasheet" " ~"
+		(property "Datasheet" "~"
 			(at 252.73 44.45 0)
 			(effects
@@
 			)
 		)
+		(property "LCSC Part #" "C426221"
+			(at 252.73 44.45 0)
+			(effects
+				(font
+					(size 1.27 1.27)
+				)
+				(hide yes)
+			)
+		)
+		(property "LCSC Part # (backup)" "C141880"
+			(at 252.73 44.45 0)
+			(effects
+				(font
+					(size 1.27 1.27)
+				)
+				(hide yes)
+			)
+		)
 		(pin "0"
 		)
@@
 			(project "pico_expansion_board"
 				(path "/b8f3f05d-f7a7-4c52-a258-9c2fea48c789/c872847a-864f-4ac1-95f5-557947400505"
-					(reference "J9")
+					(reference "J10")
 					(unit 1)
 				)
@@
 		(dnp no)
 		(fields_autoplaced yes)
-		(property "Reference" "C13"
+		(property "Reference" "C12"
 			(at 114.3 50.8 0)
 			(effects
@@
 			)
 		)
+		(property "LCSC Part #" "C49678"
+			(at 110.49 52.07 0)
+			(effects
+				(font
+					(size 1.27 1.27)
+				)
+				(hide yes)
+			)
+		)
 		(pin "1"
 		)
@@
 			(project "pico_expansion_board"
 				(path "/b8f3f05d-f7a7-4c52-a258-9c2fea48c789/c872847a-864f-4ac1-95f5-557947400505"
-					(reference "C13")
+					(reference "C12")
 					(unit 1)
 				)
@@
 		(dnp no)
 		(fields_autoplaced yes)
-		(property "Reference" "#PWR043"
+		(property "Reference" "#PWR063"
 			(at 166.37 106.68 0)
 			(effects
@@
 			(project "pico_expansion_board"
 				(path "/b8f3f05d-f7a7-4c52-a258-9c2fea48c789/c872847a-864f-4ac1-95f5-557947400505"
-					(reference "#PWR043")
+					(reference "#PWR063")
 					(unit 1)
 				)
@@
 		(dnp no)
 		(fields_autoplaced yes)
-		(property "Reference" "#PWR055"
+		(property "Reference" "#PWR065"
 			(at 252.73 69.85 0)
 			(effects
@@
 			(project "pico_expansion_board"
 				(path "/b8f3f05d-f7a7-4c52-a258-9c2fea48c789/c872847a-864f-4ac1-95f5-557947400505"
-					(reference "#PWR055")
+					(reference "#PWR065")
 					(unit 1)
 				)
@@
 		(dnp no)
 		(fields_autoplaced yes)
-		(property "Reference" "C12"
+		(property "Reference" "C11"
 			(at 72.39 35.7632 0)
 			(effects
@@
 			)
 		)
+		(property "LCSC Part #" "C49678"
+			(at 69.85 36.83 0)
+			(effects
+				(font
+					(size 1.27 1.27)
+				)
+				(hide yes)
+			)
+		)
 		(pin "1"
 		)
@@
 			(project "pico_expansion_board"
 				(path "/b8f3f05d-f7a7-4c52-a258-9c2fea48c789/c872847a-864f-4ac1-95f5-557947400505"
-					(reference "C12")
+					(reference "C11")
 					(unit 1)
 				)
@@
 			)
 		)
+		(property "LCSC Part #" "C965817"
+			(at 201.93 116.84 90)
+			(effects
+				(font
+					(size 1.27 1.27)
+				)
+				(hide yes)
+			)
+		)
 		(pin "1"
 		)
@@
 		(dnp no)
 		(fields_autoplaced yes)
-		(property "Reference" "C15"
+		(property "Reference" "C14"
 			(at 121.285 54.61 90)
 			(effects
@@
 			)
 		)
+		(property "LCSC Part #" "C49678"
+			(at 121.92 60.96 90)
+			(effects
+				(font
+					(size 1.27 1.27)
+				)
+				(hide yes)
+			)
+		)
 		(pin "1"
 		)
@@
 			(project "pico_expansion_board"
 				(path "/b8f3f05d-f7a7-4c52-a258-9c2fea48c789/c872847a-864f-4ac1-95f5-557947400505"
-					(reference "C15")
+					(reference "C14")
 					(unit 1)
 				)
@@
 		(dnp no)
 		(fields_autoplaced yes)
-		(property "Reference" "#PWR050"
+		(property "Reference" "#PWR058"
 			(at 69.85 45.72 0)
 			(effects
@@
 			(project "pico_expansion_board"
 				(path "/b8f3f05d-f7a7-4c52-a258-9c2fea48c789/c872847a-864f-4ac1-95f5-557947400505"
-					(reference "#PWR050")
+					(reference "#PWR058")
 					(unit 1)
 				)
@@
 		(on_board yes)
 		(dnp no)
-		(property "Reference" "R13"
+		(property "Reference" "R11"
 			(at 171.45 105.41 0)
 			(effects
@@
 			)
 		)
+		(property "LCSC Part #" "C17513"
+			(at 166.37 106.68 0)
+			(effects
+				(font
+					(size 1.27 1.27)
+				)
+				(hide yes)
+			)
+		)
 		(pin "1"
 		)
@@
 			(project "pico_expansion_board"
 				(path "/b8f3f05d-f7a7-4c52-a258-9c2fea48c789/c872847a-864f-4ac1-95f5-557947400505"
-					(reference "R13")
+					(reference "R11")
 					(unit 1)
 				)
@@
 		(dnp no)
 		(fields_autoplaced yes)
-		(property "Reference" "#PWR054"
+		(property "Reference" "#PWR062"
 			(at 135.89 60.96 0)
 			(effects
@@
 			(project "pico_expansion_board"
 				(path "/b8f3f05d-f7a7-4c52-a258-9c2fea48c789/c872847a-864f-4ac1-95f5-557947400505"
-					(reference "#PWR054")
+					(reference "#PWR062")
 					(unit 1)
 				)
@@
 		(dnp no)
 		(fields_autoplaced yes)
-		(property "Reference" "J8"
+		(property "Reference" "J9"
 			(at 177.8 31.75 0)
 			(effects
@@
 			)
 		)
+		(property "LCSC Part #" "C2935957"
+			(at 176.53 38.1 0)
+			(effects
+				(font
+					(size 1.27 1.27)
+				)
+				(hide yes)
+			)
+		)
+		(property "LCSC Part # (backup)" "C2905988"
+			(at 176.53 38.1 0)
+			(effects
+				(font
+					(size 1.27 1.27)
+				)
+				(hide yes)
+			)
+		)
 		(pin "2"
 		)
@@
 			(project ""
 				(path "/b8f3f05d-f7a7-4c52-a258-9c2fea48c789/c872847a-864f-4ac1-95f5-557947400505"
-					(reference "J8")
+					(reference "J9")
 					(unit 1)
 				)
@@
 			)
 		)
+		(property "LCSC Part #" "C84256"
+			(at 166.37 116.84 90)
+			(effects
+				(font
+					(size 1.27 1.27)
+				)
+				(hide yes)
+			)
+		)
 		(pin "1"
 		)
@@
 		(dnp no)
 		(fields_autoplaced yes)
-		(property "Reference" "#PWR041"
+		(property "Reference" "#PWR064"
 			(at 201.93 106.68 0)
 			(effects
@@
 			(project "pico_expansion_board"
 				(path "/b8f3f05d-f7a7-4c52-a258-9c2fea48c789/c872847a-864f-4ac1-95f5-557947400505"
-					(reference "#PWR041")
+					(reference "#PWR064")
 					(unit 1)
 				)
@@
 		(dnp no)
 		(fields_autoplaced yes)
-		(property "Reference" "C14"
+		(property "Reference" "C13"
 			(at 112.395 62.23 90)
 			(effects
@@
 			)
 		)
+		(property "LCSC Part #" "C49678"
+			(at 111.76 68.58 90)
+			(effects
+				(font
+					(size 1.27 1.27)
+				)
+				(hide yes)
+			)
+		)
 		(pin "1"
 		)
@@
 			(project "pico_expansion_board"
 				(path "/b8f3f05d-f7a7-4c52-a258-9c2fea48c789/c872847a-864f-4ac1-95f5-557947400505"
-					(reference "C14")
-					(unit 1)
-				)
+					(reference "C13")
+					(unit 1)
+				)

Commit message: Add production files with placements
Parts:
- J10: JLCPCB Position Offset (none) -> 0,5.9055
Changed lines of the file:
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@@
+			)
+		)
+		(property "JLCPCB Position Offset" "0,5.9055"
+			(at 252.73 44.45 0)
+			(effects
+				(font
+					(size 1.27 1.27)
+				)
+				(hide yes)
 			)
 		)
